File: design_files/ASM2021.sch (EAGLE design)
At the start: 40 parts, among them J1 47346-0001, J2 SM02B-SRSS, J3 961102, J6 DF12-32-DP, Q1 DMP2035U, SW1 PCM12SMTR, SW2 KMT011, U1 XC6210B33, U2 MCP73831, U3 ATSAMD21G18A, U4 BMA250, Y1 32.7680

Commit message: Update ASM2021.sch
Parts:
- removed J7: (no value), tinycircuits:TEST_POINT
- U4: value BMA250 -> BMA250E
Connections:
- net AD4 renamed AD4(VBATT_DIV)
- net AD4/SDA renamed SDA
- net AD5/SCL renamed SCL
- removed net AD5: SW2.2, U3.PB02
- removed net ATN/IO38: U3.PA13
- removed net MISO_ALT: U3.PA12
- removed net MOSI_ALT: U3.PB10
- removed net RX_LED/IO27/AIN11: U3.PB03
- removed net SCK_ALT: U3.PB11
- removed net TX_LED/IO26: U3.PA27
- removed net USB_HOST_EN/IO27: U3.PA28
- new net AD5(BOOTLOADER): SW2.2
- new net AD5(BOOT_SW): U3.PB02
- net GND: now also R9.1, SW1.3
- net INT1: no longer J7.1
- net SWDIO: no longer R9.1, U3.PA31
- net VCC: now also U4.SDO
Other:
- note added: "5"
- note added: "BMA250E Accelerometer"
- note added: "Non Populated: -"
- note added: "Non Populated: U4"
- note added: "Variant: Accelerometer - R-A"
- note removed: "4"
- note removed: "BMA250 Accelerometer"
- note removed: "Non Populated: C12, U4"
- moved on the sheet: C12, C5, C6, Y1
