File: design_files/ASM2021.brd (EAGLE design)
At the start: 22.5 x 21.3 mm, 41 parts, among them J1 47346-0001, J2 SM02B-SRSS, J3 961102, J6 DF12-32-DP, Q1 DMP2035U, SW1 PCM12SMTR, SW2 KMT011, U1 XC6210B33, U2 MCP73831, U3 ATSAMD21G18A, U4 BMA250, Y1 32.7680

Commit message: Update ASM2021.brd
Parts:
- removed J7: (no value), tinycircuits:TEST_POINT_1MM
- U4: value BMA250 -> BMA250E
- moved R9 0.25 mm to (26.1, 19.4)
Connections:
- net AD4 renamed AD4(VBATT_DIV)
- net AD4/SDA renamed SDA
- net AD5/SCL renamed SCL
- removed net AD5: SW2.2, U3.47
- removed net ATN/IO38: U3.22
- removed net MISO_ALT: U3.21
- removed net MOSI_ALT: U3.19
- removed net RX_LED/IO27/AIN11: U3.48
- removed net SCK_ALT: U3.20
- removed net TX_LED/IO26: U3.39
- removed net USB_HOST_EN/IO27: U3.41
- new net AD5(BOOTLOADER): SW2.2
- new net AD5(BOOT_SW): U3.47
- net GND: now also R9.1, SW1.3
- net INT1: no longer J7.P$1
- net SWDIO: no longer R9.1, U3.46
- net VCC: now also U4.1
Routing:
- net AD5: track 10.1 -> 0.00 mm
- net AD5(BOOTLOADER): track 0.00 -> 8.11 mm
- net SWDIO: track 33.8 -> 32.0 mm, vias 2 -> 1
- net VCC: track 82.6 -> 84.0 mm, vias 4 -> 5
- net INT1: track 1.81 -> 3.18 mm
- net GND: vias 17 -> 18
Other:
- board text added: "5"
- board text added: "ASM2021 Rev5"
- board text removed: "4"
- board text removed: "ASM2021 Rev4"
